File: Electronics/PianoKeychain.kicad_pcb (KiCad board)
At the start: 2 copper layers, 86.4 x 31.9 mm, 24 parts, among them SW1 1825910-6, SW2 1825910-6, SW3 1825910-6, SW4 1825910-6, SW5 1825910-6, SW6 1825910-6, SW7 1825910-6, SW8 1825910-6, U1 LM555xN

Commit message: Updated case 3d model to exclude key ring, changed silkscreen
Parts:
- renumbered LS1 to Speaker
Changed lines of the file:
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@@
     (property "Sheetname" "")
     (attr through_hole)
-    (fp_text reference "LS1" (at 10.936043 -7.574222) (layer "F.SilkS")
+    (fp_text reference "Speaker" (at 10.936043 -7.574222) (layer "F.SilkS")
       (effects (font (size 1 1) (thickness 0.15)))
     )
